File: LK3000_Keyboard/LK3000_Keyboard.kicad_sch (KiCad schematic)
At the start: 34 parts, among them J1 Keyboard, SW1 A [MET], SW10 T [+/-], SW11 U [M+], SW12 V [0], SW13 E [7], SW14 F [8], SW15 G [9], SW16 H [÷], SW17 N [4], SW18 O [5], SW19 P [6], SW2 B [US], SW20 Q [+], SW21 W [1], SW22 X [2], SW23 Y [3], SW24 Z [.], SW25 ? [P2}, SW26 bs [P1], SW27 R [-], SW28 I [x], SW29 def [P4], SW3 C [X->M], SW30 stp [P3], SW31 sp [=], SW32 f, SW33 clr, SW4 D [K], SW5 J [C1], SW6 K [C2], SW7 L [RM], SW8 M [%], SW9 S [EXC]

Commit message: Revised keyboard design to use 12mm tactile
Parts:
- SW1, SW10, SW11, SW12, SW13, SW14, SW15, SW16, SW17, SW18, SW19, SW2, SW20, SW21, SW22, SW23, SW24, SW25, SW26, SW27, SW28, SW29, SW3, SW30, SW31, SW32, SW33, SW4, SW5, SW6, SW7, SW8, SW9: footprint Clueless_Engineer:SW_Gateron_LowProfile_THT -> Button_Switch_THT:SW_PUSH-12mm_Wuerth-430476085716
Other:
- title: Nixdorf LK-3000 Keyboard -> Nixdorf LK-3000 Development Keyboard
Changed lines of the file:
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@@
 	(paper "A4")
 	(title_block
-		(title "Nixdorf LK-3000 Keyboard")
+		(title "Nixdorf LK-3000 Development Keyboard")
 		(date "24/SEP/2025")
 		(rev "A")
@@
 			)
 		)
-		(property "Footprint" "Clueless_Engineer:SW_Gateron_LowProfile_THT"
+		(property "Footprint" "Button_Switch_THT:SW_PUSH-12mm_Wuerth-430476085716"
 			(at 146.05 55.88 0)
 			(effects
@@
 			)
 		)
-		(property "Footprint" "Clueless_Engineer:SW_Gateron_LowProfile_THT"
+		(property "Footprint" "Button_Switch_THT:SW_PUSH-12mm_Wuerth-430476085716"
 			(at 115.57 135.89 0)
 			(effects
@@
 			)
 		)
-		(property "Footprint" "Clueless_Engineer:SW_Gateron_LowProfile_THT"
+		(property "Footprint" "Button_Switch_THT:SW_PUSH-12mm_Wuerth-430476085716"
 			(at 130.81 95.25 0)
 			(effects
@@
 			)
 		)
-		(property "Footprint" "Clueless_Engineer:SW_Gateron_LowProfile_THT"
+		(property "Footprint" "Button_Switch_THT:SW_PUSH-12mm_Wuerth-430476085716"
 			(at 115.57 151.13 0)
 			(effects
@@
 			)
 		)
-		(property "Footprint" "Clueless_Engineer:SW_Gateron_LowProfile_THT"
+		(property "Footprint" "Button_Switch_THT:SW_PUSH-12mm_Wuerth-430476085716"
 			(at 100.33 151.13 0)
 			(effects
@@
 			)
 		)
-		(property "Footprint" "Clueless_Engineer:SW_Gateron_LowProfile_THT"
+		(property "Footprint" "Button_Switch_THT:SW_PUSH-12mm_Wuerth-430476085716"
 			(at 146.05 135.89 0)
 			(effects
@@
 			)
 		)
-		(property "Footprint" "Clueless_Engineer:SW_Gateron_LowProfile_THT"
+		(property "Footprint" "Button_Switch_THT:SW_PUSH-12mm_Wuerth-430476085716"
 			(at 100.33 82.55 0)
 			(effects
@@
 			)
 		)
-		(property "Footprint" "Clueless_Engineer:SW_Gateron_LowProfile_THT"
+		(property "Footprint" "Button_Switch_THT:SW_PUSH-12mm_Wuerth-430476085716"
 			(at 146.05 82.55 0)
 			(effects
@@
 			)
 		)
-		(property "Footprint" "Clueless_Engineer:SW_Gateron_LowProfile_THT"
+		(property "Footprint" "Button_Switch_THT:SW_PUSH-12mm_Wuerth-430476085716"
 			(at 100.33 68.58 0)
 			(effects
@@
 			)
 		)
-		(property "Footprint" "Clueless_Engineer:SW_Gateron_LowProfile_THT"
+		(property "Footprint" "Button_Switch_THT:SW_PUSH-12mm_Wuerth-430476085716"
 			(at 100.33 107.95 0)
 			(effects
@@
 			)
 		)
-		(property "Footprint" "Clueless_Engineer:SW_Gateron_LowProfile_THT"
+		(property "Footprint" "Button_Switch_THT:SW_PUSH-12mm_Wuerth-430476085716"
 			(at 130.81 55.88 0)
 			(effects
@@
 			)
 		)
-		(property "Footprint" "Clueless_Engineer:SW_Gateron_LowProfile_THT"
+		(property "Footprint" "Button_Switch_THT:SW_PUSH-12mm_Wuerth-430476085716"
 			(at 115.57 82.55 0)
 			(effects
@@
 			)
 		)
-		(property "Footprint" "Clueless_Engineer:SW_Gateron_LowProfile_THT"
+		(property "Footprint" "Button_Switch_THT:SW_PUSH-12mm_Wuerth-430476085716"
 			(at 146.05 151.13 0)
 			(effects
@@
 			)
 		)
-		(property "Footprint" "Clueless_Engineer:SW_Gateron_LowProfile_THT"
+		(property "Footprint" "Button_Switch_THT:SW_PUSH-12mm_Wuerth-430476085716"
 			(at 130.81 120.65 0)
 			(effects
@@
 			)
 		)
-		(property "Footprint" "Clueless_Engineer:SW_Gateron_LowProfile_THT"
+		(property "Footprint" "Button_Switch_THT:SW_PUSH-12mm_Wuerth-430476085716"
 			(at 130.81 68.58 0)
 			(effects
@@
 			)
 		)
-		(property "Footprint" "Clueless_Engineer:SW_Gateron_LowProfile_THT"
+		(property "Footprint" "Button_Switch_THT:SW_PUSH-12mm_Wuerth-430476085716"
 			(at 130.81 151.13 0)
 			(effects
@@
 			)
 		)
-		(property "Footprint" "Clueless_Engineer:SW_Gateron_LowProfile_THT"
+		(property "Footprint" "Button_Switch_THT:SW_PUSH-12mm_Wuerth-430476085716"
 			(at 130.81 107.95 0)
 			(effects
@@
 			)
 		)
-		(property "Footprint" "Clueless_Engineer:SW_Gateron_LowProfile_THT"
+		(property "Footprint" "Button_Switch_THT:SW_PUSH-12mm_Wuerth-430476085716"
 			(at 100.33 55.88 0)
 			(effects
@@
 			)
 		)
-		(property "Footprint" "Clueless_Engineer:SW_Gateron_LowProfile_THT"
+		(property "Footprint" "Button_Switch_THT:SW_PUSH-12mm_Wuerth-430476085716"
 			(at 100.33 95.25 0)
 			(effects
@@
 			)
 		)
-		(property "Footprint" "Clueless_Engineer:SW_Gateron_LowProfile_THT"
+		(property "Footprint" "Button_Switch_THT:SW_PUSH-12mm_Wuerth-430476085716"
 			(at 115.57 55.88 0)
 			(effects
@@
 			)
 		)
-		(property "Footprint" "Clueless_Engineer:SW_Gateron_LowProfile_THT"
+		(property "Footprint" "Button_Switch_THT:SW_PUSH-12mm_Wuerth-430476085716"
 			(at 100.33 120.65 0)
 			(effects
@@
 			)
 		)
-		(property "Footprint" "Clueless_Engineer:SW_Gateron_LowProfile_THT"
+		(property "Footprint" "Button_Switch_THT:SW_PUSH-12mm_Wuerth-430476085716"
 			(at 146.05 95.25 0)
 			(effects
@@
 			)
 		)
-		(property "Footprint" "Clueless_Engineer:SW_Gateron_LowProfile_THT"
+		(property "Footprint" "Button_Switch_THT:SW_PUSH-12mm_Wuerth-430476085716"
 			(at 130.81 135.89 0)
 			(effects
@@
 			)
 		)
-		(property "Footprint" "Clueless_Engineer:SW_Gateron_LowProfile_THT"
+		(property "Footprint" "Button_Switch_THT:SW_PUSH-12mm_Wuerth-430476085716"
 			(at 115.57 107.95 0)
 			(effects
@@
 			)
 		)
-		(property "Footprint" "Clueless_Engineer:SW_Gateron_LowProfile_THT"
+		(property "Footprint" "Button_Switch_THT:SW_PUSH-12mm_Wuerth-430476085716"
 			(at 196.85 114.3 0)
 			(effects
@@
 			)
 		)
-		(property "Footprint" "Clueless_Engineer:SW_Gateron_LowProfile_THT"
+		(property "Footprint" "Button_Switch_THT:SW_PUSH-12mm_Wuerth-430476085716"
 			(at 115.57 120.65 0)
 			(effects
@@
 			)
 		)
-		(property "Footprint" "Clueless_Engineer:SW_Gateron_LowProfile_THT"
+		(property "Footprint" "Button_Switch_THT:SW_PUSH-12mm_Wuerth-430476085716"
 			(at 130.81 82.55 0)
 			(effects
@@
 			)
 		)
-		(property "Footprint" "Clueless_Engineer:SW_Gateron_LowProfile_THT"
+		(property "Footprint" "Button_Switch_THT:SW_PUSH-12mm_Wuerth-430476085716"
 			(at 115.57 68.58 0)
 			(effects
@@
 			)
 		)
-		(property "Footprint" "Clueless_Engineer:SW_Gateron_LowProfile_THT"
+		(property "Footprint" "Button_Switch_THT:SW_PUSH-12mm_Wuerth-430476085716"
 			(at 100.33 135.89 0)
 			(effects
@@
 			)
 		)
-		(property "Footprint" "Clueless_Engineer:SW_Gateron_LowProfile_THT"
+		(property "Footprint" "Button_Switch_THT:SW_PUSH-12mm_Wuerth-430476085716"
 			(at 146.05 107.95 0)
 			(effects
@@
 			)
 		)
-		(property "Footprint" "Clueless_Engineer:SW_Gateron_LowProfile_THT"
+		(property "Footprint" "Button_Switch_THT:SW_PUSH-12mm_Wuerth-430476085716"
 			(at 115.57 95.25 0)
 			(effects
@@
 			)
 		)
-		(property "Footprint" "Clueless_Engineer:SW_Gateron_LowProfile_THT"
+		(property "Footprint" "Button_Switch_THT:SW_PUSH-12mm_Wuerth-430476085716"
 			(at 146.05 68.58 0)
 			(effects
@@
 			)
 		)
-		(property "Footprint" "Clueless_Engineer:SW_Gateron_LowProfile_THT"
+		(property "Footprint" "Button_Switch_THT:SW_PUSH-12mm_Wuerth-430476085716"
 			(at 146.05 120.65 0)
 			(effects
